File: Kicad_Project_Files/ESC_indev_undergoing.kicad_pcb (KiCad board)
At the start: 2 copper layers, 39 parts, among them J1 XT60-M, Q1 NMOS, Q2 NMOS, Q3 NMOS, Q4 NMOS, Q5 NMOS, Q6 NMOS, SW1 SW_Push, U2 IR2110, U3 IR2110, U4 IR2110, U5 ESP32-WROOM-32E

Commit message: major pcb desgin advance
Parts:
- removed J1: XT60-M, Connector_AMASS:AMASS_XT60PW-M_1x02_P7.20mm_Horizontal
- added C1: C, Capacitor_SMD:C_1206_3216Metric, F.Cu at (250.1, 86.0)
- added D4: LED, LED_SMD:LED_0603_1608Metric_Pad1.05x0.95mm_HandSolder, F.Cu at (167.0, 68.1)
- added J2: JST_PH_1x04_P2mm, PCM_fab:Header_JST_PH_1x04_P2mm_Vertical_SMD, F.Cu at (228.0, 34.5)
- added J3: JST_PH_1x04_P2mm, PCM_fab:Header_JST_PH_1x04_P2mm_Vertical_SMD, F.Cu at (213.5, 34.5)
- added R16: 33k, PCM_Resistor_SMD_AKL:R_0603_1608Metric_Pad1.05x0.95mm_HandSolder, F.Cu at (175.2, 59.8)
- added R17: 33k, PCM_Resistor_SMD_AKL:R_0603_1608Metric_Pad1.05x0.95mm_HandSolder, F.Cu at (168.7, 75.8)
- added R18: 10k, PCM_Resistor_SMD_AKL:R_0603_1608Metric_Pad1.05x0.95mm_HandSolder, F.Cu at (168.7, 78.3)
- added R19: 33k, PCM_Resistor_SMD_AKL:R_0603_1608Metric_Pad1.05x0.95mm_HandSolder, F.Cu at (168.7, 80.8)
- added R20: 10k, PCM_Resistor_SMD_AKL:R_0603_1608Metric_Pad1.05x0.95mm_HandSolder, F.Cu at (168.7, 83.3)
- added R21: 33k, PCM_Resistor_SMD_AKL:R_0603_1608Metric_Pad1.05x0.95mm_HandSolder, F.Cu at (168.7, 85.8)
- added R22: 33k, PCM_Resistor_SMD_AKL:R_0603_1608Metric_Pad1.05x0.95mm_HandSolder, F.Cu at (168.7, 88.3)
- added R23: 10k, PCM_Resistor_SMD_AKL:R_0603_1608Metric_Pad1.05x0.95mm_HandSolder, F.Cu at (168.7, 90.9)
- added R24: 33k, PCM_Resistor_SMD_AKL:R_0603_1608Metric_Pad1.05x0.95mm_HandSolder, F.Cu at (168.7, 93.4)
- added R25: 10k, PCM_Resistor_SMD_AKL:R_0603_1608Metric_Pad1.05x0.95mm_HandSolder, F.Cu at (175.2, 62.3)
- added SW2: SW_Push, Button_Switch_SMD:SW_Push_1P1T_NO_CK_KMR2, F.Cu at (229.6, 54.0)
- added U1: TPS560430X3FDBVR, Kicad_Project_Files:IC_TPS560430X3FDBVR, B.Cu at (201.5, 49.2)
- added U10: ~, solderpads:Untitled, F.Cu at (187.8, 69.2)
- added U11: LMV324, PCM_Package_SO_AKL:SSOP-14_5.3x6.2mm_P0.65mm, F.Cu at (175.9, 78.6)
- added U6: ~, solderpads:Untitled, B.Cu at (210.0, 104.5)
- added U7: ~, solderpads:Untitled, B.Cu at (227.5, 104.5)
- added U8: ~, solderpads:Untitled, B.Cu at (244.0, 105.2)
- added U9: ~, solderpads:Untitled, F.Cu at (188.0, 58.8)
- C4, C5, C6: footprint Capacitor_SMD:C_1206_3216Metric -> Capacitor_SMD:C_0805_2012Metric
- C7, C8, C9, L1: moved to B.Cu
- D1, D2, D3: footprint Diode_THT:D_DO-41_SOD81_P10.16mm_Horizontal -> Diode_SMD:D_1206_3216Metric_Pad1.42x1.75mm_HandSolder
- Q1, Q2, Q3, Q4, Q5, Q6: footprint PCM_Package_TO_SOT_THT_AKL:TO-220-3_Horizontal_TabDown -> Kicad_Project_Files:TO-263-2; moved to B.Cu
- R1, R6, R7: footprint PCM_Resistor_SMD_AKL:R_1206_3216Metric -> PCM_Resistor_SMD_AKL:R_0603_1608Metric_Pad1.05x0.95mm_HandSolder
- R10, R11, R14, R15, R2, R3: footprint PCM_Resistor_SMD_AKL:R_1206_3216Metric -> PCM_Resistor_SMD_AKL:R_0603_1608Metric_Pad1.05x0.95mm_HandSolder; moved to B.Cu
- R12, R4, R5, R8: value R_US -> 10k; footprint PCM_Resistor_SMD_AKL:R_1206_3216Metric -> PCM_Resistor_SMD_AKL:R_0603_1608Metric_Pad1.05x0.95mm_HandSolder; moved to B.Cu
- R13, R9: value R_US -> 10k; footprint PCM_Resistor_SMD_AKL:R_1206_3216Metric -> PCM_Resistor_SMD_AKL:R_0603_1608Metric_Pad1.05x0.95mm_HandSolder
- U2, U3, U4: value IR2110 -> IR2110S; footprint Package_DIP:DIP-14_W7.62mm -> Package_SO:SOIC-16W_7.5x10.3mm_P1.27mm
- moved U5 154.9 mm to (249.3, 50.0), turned to -90 degrees
- moved U2 119.0 mm to (242.9, 88.7)
- moved D1 113.3 mm to (252.5, 88.2), turned to -90 degrees
- moved C6 112.8 mm to (250.3, 91.0), turned to -90 degrees
- moved R4 108.0 mm to (244.5, 81.3)
- moved R2 106.9 mm to (244.4, 82.8)
- moved R5 102.3 mm to (238.0, 81.5), turned to 90 degrees
- moved R3 101.5 mm to (238.0, 78.6), turned to -90 degrees
- moved SW1 96.3 mm to (229.2, 42.5), turned to 90 degrees
- moved C2 95.2 mm to (230.0, 86.3), turned to -90 degrees
- moved C4 94.7 mm to (230.0, 91.5), turned to -90 degrees
- moved D2 93.6 mm to (232.5, 89.1), turned to -90 degrees
- moved U3 93.4 mm to (222.8, 88.4)
- moved R7 91.0 mm to (234.5, 95.2)
- moved R9 90.3 mm to (234.0, 93.0), turned to 180 degrees
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Connections:
- net +15V renamed /15v
- C2 pad 2: /Vs2 -> /P2
- C3 pad 2: /Vs3 -> /P3
- Q1 pad 3: /Vs1 -> /P1
- Q2 pad 1: /Vs1 -> /P1
- Q3 pad 3: /Vs2 -> /P2
- Q4 pad 1: /Vs2 -> /P2
- Q5 pad 3: /Vs3 -> /P3
- Q6 pad 1: /Vs3 -> /P3
- R12 pad 1: GND -> /P3
- R4 pad 1: GND -> /P1
- R8 pad 1: GND -> /P2
- U2 pad 10: /HIN1 -> unconnected-(U2-NC-Pad10)
- U2 pad 11: GND -> +3.3V
- U2 pad 12: /LIN1 -> /HIN1
- U2 pad 14: unconnected-(U2-NC-Pad14) -> /LIN1
- U2 pad 5: /Vs1 -> unconnected-(U2-NC-Pad5)
- U2 pad 6: Net-(D1-K) -> /P1
- U2 pad 7: /HO1 -> Net-(D1-K)
- U2 pad 8: unconnected-(U2-NC-Pad8) -> /HO1
- U2 pad 9: +3.3V -> unconnected-(U2-NC-Pad9)
- U3 pad 10: /HIN2 -> unconnected-(U3-NC-Pad10)
- U3 pad 11: GND -> +3.3V
- U3 pad 12: /LIN2 -> /HIN2
- U3 pad 14: unconnected-(U3-NC-Pad14) -> /LIN2
- U3 pad 5: /Vs2 -> unconnected-(U3-NC-Pad5)
- U3 pad 6: Net-(D2-K) -> /P2
- U3 pad 7: /HO2 -> Net-(D2-K)
- U3 pad 8: unconnected-(U3-NC-Pad8) -> /HO2
- U3 pad 9: +3.3V -> unconnected-(U3-NC-Pad9)
- U4 pad 10: /HIN3 -> unconnected-(U4-NC-Pad10)
- U4 pad 11: GND -> +3.3V
- U4 pad 12: /LIN3 -> /HIN3
- U4 pad 14: unconnected-(U4-NC-Pad14) -> /LIN3
- U4 pad 5: /Vs3 -> unconnected-(U4-NC-Pad5)
- U4 pad 6: Net-(D3-K) -> /P3
- U4 pad 7: /HO3 -> Net-(D3-K)
- U4 pad 8: unconnected-(U4-NC-Pad8) -> /HO3
- U5 pad 25: unconnected-(U5-IO0-Pad25) -> Net-(U5-IO0)
- U5 pad 33: unconnected-(U5-IO21-Pad33) -> Net-(U5-IO21)
- U5 pad 34: unconnected-(U5-RXD0/IO3-Pad34) -> Net-(U5-RXD0/IO3)
- U5 pad 35: unconnected-(U5-TXD0/IO1-Pad35) -> Net-(U5-TXD0/IO1)
- U5 pad 36: unconnected-(U5-IO22-Pad36) -> Net-(U5-IO22)
Routing:
- net /LIN3: track 0.00 -> 117.3 mm
- net /HIN3: track 0.00 -> 112.8 mm
- net /LIN2: track 0.00 -> 94.4 mm
- net /HIN2: track 0.00 -> 92.6 mm
- net /LIN1: track 0.00 -> 74.1 mm
- net /HIN1: track 0.00 -> 70.4 mm
- net Net-(U5-IO21): track 0.00 -> 60.6 mm, vias 0 -> 2
- net Net-(U5-IO22): track 0.00 -> 58.8 mm, vias 0 -> 2
- net Net-(U5-TXD0/IO1): track 0.00 -> 38.6 mm
- net Net-(U5-RXD0/IO3): track 0.00 -> 37.2 mm, vias 0 -> 2
- net Net-(Q4-G): track 0.00 -> 20.1 mm
- net /LO3: track 0.00 -> 19.3 mm
- net /LO1: track 0.00 -> 16.7 mm
- net GND: track 0.00 -> 15.6 mm, vias 0 -> 6
- net /15v: track 0.00 -> 13.9 mm, vias 0 -> 63
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- added copper zone on F.Cu, net /15v
- added copper zone on B.Cu, net /P1
- added copper zone on B.Cu, net /P2
- added copper zone on B.Cu, net /P3
- added copper zone on B.Cu, net GND
- added copper zone on F.Cu, net GND
Other:
- board outline added: 64.5 x 76.5 mm

Commit message: added traces to drivers
Parts:
- added H1: MountingHole_Pad, MountingHole:MountingHole_3.2mm_M3_DIN965_Pad, F.Cu at (199.0, 34.0)
- added H2: MountingHole_Pad, MountingHole:MountingHole_3.2mm_M3_DIN965_Pad, F.Cu at (251.0, 34.0)
- added H3: MountingHole_Pad, MountingHole:MountingHole_3.2mm_M3_DIN965_Pad, F.Cu at (251.0, 101.0)
- added H4: MountingHole_Pad, MountingHole:MountingHole_3.2mm_M3_DIN965_Pad, F.Cu at (199.0, 101.0)
- D4, R16, R17, R18, R19, R20, R21, R22, R23, R24, R6: moved to B.Cu
- R2, R3, R4: moved to F.Cu
- U11: footprint PCM_Package_SO_AKL:SSOP-14_5.3x6.2mm_P0.65mm -> PCM_Package_SO_AKL:SOIC-14_3.9x8.7mm_P1.27mm; moved to B.Cu
- moved R17 79.2 mm to (246.0, 58.5)
- moved R19 66.8 mm to (231.5, 58.0), turned to -90 degrees
- moved R20 64.6 mm to (226.5, 54.5), turned to -90 degrees
- moved R21 63.7 mm to (225.5, 57.0), turned to 180 degrees
- moved R23 59.4 mm to (217.9, 57.5)
- moved R24 57.2 mm to (213.5, 57.9), turned to 90 degrees
- moved R22 56.7 mm to (217.9, 60.0), turned to 180 degrees
- moved R25 56.6 mm to (230.0, 48.0), turned to 90 degrees
- moved R1 53.2 mm to (228.0, 48.0), turned to -90 degrees
- moved R18 53.0 mm to (215.0, 52.4), turned to -90 degrees
- moved U11 52.1 mm to (221.0, 52.5), turned to 90 degrees
- moved R6 50.9 mm to (220.5, 80.5), turned to 90 degrees
- moved D4 46.4 mm to (208.0, 46.5), turned to -90 degrees
- moved R16 39.9 mm to (215.0, 56.4), turned to -90 degrees
- moved R10 26.1 mm to (201.5, 84.5), turned to 90 degrees
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Connections:
- U11 pad 1: unconnected-(U11-Pad1) -> Net-(U5-IO26)
- U11 pad 7: unconnected-(U11-Pad7) -> Net-(U5-IO27)
- U11 pad 8: unconnected-(U11-Pad8) -> Net-(U5-IO32)
- U5 pad 11: unconnected-(U5-IO26-Pad11) -> Net-(U5-IO26)
- U5 pad 12: unconnected-(U5-IO27-Pad12) -> Net-(U5-IO27)
- U5 pad 8: unconnected-(U5-IO32-Pad8) -> Net-(U5-IO32)
Routing:
- net +3.3V: track 0.48 -> 77.5 mm, vias 0 -> 4
- net Net-(U11C-+): track 0.00 -> 38.6 mm
- net Net-(Q1-G): track 0.00 -> 35.7 mm, vias 0 -> 1
- net Net-(Q5-G): track 7.13 -> 29.3 mm
- net Net-(Q3-G): track 3.99 -> 23.1 mm
- net Net-(U1-FB): track 0.00 -> 16.4 mm
- net Net-(U11B-+): track 0.00 -> 15.8 mm
- net Net-(Q6-G): track 4.35 -> 19.5 mm
- net /P3: track 7.44 -> 22.5 mm, vias 0 -> 1
- net /LO3: track 19.3 -> 4.84 mm, vias 0 -> 1
- net Net-(U11A-+): track 0.00 -> 13.4 mm
- net Net-(Q2-G): track 9.12 -> 21.8 mm, vias 0 -> 1
- net Net-(U1-SW): track 0.00 -> 11.4 mm
- net Net-(U1-CB): track 0.00 -> 10.2 mm
- net /HO2: track 0.00 -> 9.25 mm, vias 0 -> 1
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- added copper zone on B.Cu, net +3.3V

Commit message: driver trace update
Parts:
- moved R6 0.50 mm to (220.0, 80.5)
Routing:
- net /15v: track 17.5 -> 89.9 mm, vias 63 -> 66
- net /HO2: track 9.25 -> 13.4 mm
- net GND: track 15.7 -> 18.5 mm
- net +3.3V: track 77.5 -> 78.9 mm
- net /HO1: track 8.10 -> 8.83 mm
- net Net-(Q1-G): track 35.7 -> 36.4 mm
